Commit message: divide robot into three parts
* these three parts are:astra/kinect.urdf.xacro,
 saturnbot_base.urdf.xacro and saturnbot_gazebo.urdf.xacro
* add gitignore file
* change robot size to be like real robot

File: robot/saturnbot_astra.urdf.xacro (robot description, xacro)
@@ -3,123 +3,7 @@
     - 3d Sensor : astra
 -->
-<robot name="turtlebot" xmlns:xacro="http://ros.org/wiki/xacro">
-  <xacro:property name="length_wheel" value="0.05" />
-	<xacro:property name="radius_wheel" value="0.05" />
-	<xacro:property name="camera_link" value="0.05" />
-  <xacro:property name="M_PI" value="3.1415926535897931" />
-	<xacro:macro name="default_inertial" params="mass">
-               <inertial>
-                       <mass value="${mass}" />
-                       <inertia ixx="1.0" ixy="0.0" ixz="0.0"
-                                iyy="1.0" iyz="0.0"
-                                izz="1.0" />
-               </inertial>
-	</xacro:macro>
-  <xacro:include filename="$(find saturnbot_description)/urdf/saturnbot_properties.urdf.xacro" />
-	<link name="base_footprint">
-   		<visual>
-			<geometry>
-      				<box size="0.001 0.001 0.001"/>
-     			</geometry>
-			<origin rpy="0 0 0" xyz="0 0 0"/>
-   		</visual>
-		<!--<xacro:default_inertial mass="0.0001"/>-->
- 	</link>
-	<gazebo reference="base_footprint">
-		<material>Gazebo/Green</material>
-		<turnGravityOff>false</turnGravityOff>
-	</gazebo>
-	<joint name="base_footprint_joint" type="fixed">
-		<origin xyz="0 0 0" />
-		<parent link="base_footprint" />
-		<child link="base_link" />
-	</joint>
-	<link name="base_link">
-   		<visual>
-			<geometry>
-      				<box size="0.2 .3 .1"/>
-     			</geometry>
-			<origin rpy="0 0 1.54" xyz="0 0 0.05"/>
-			<material name="white">
-				<color rgba="1 1 1 1"/>
-			</material>
-   		</visual>
-		<collision>
-			<geometry>
-       				<box size="0.2 .3 0.1"/>
-			</geometry>
-		</collision>
-		<xacro:default_inertial mass="10"/>
- 	</link>
- 	<link name="wheel_left">
-   		<visual>
-     			<geometry>
-       				<cylinder length="${length_wheel}" radius="${radius_wheel}"/>
-     			</geometry>
-			<!-- <origin rpy="0 1.5 0" xyz="0.1 0.1 0"/> -->
-			<origin rpy="0 0 0" xyz="0 0 0"/>
-   			<material name="black">
-				<color rgba="0 0 0 1"/>
-			</material>
-		</visual>
-		<collision>
-			<geometry>
-       				<cylinder length="${length_wheel}" radius="${radius_wheel}"/>
-			</geometry>
-		</collision>
-		<xacro:default_inertial mass="1"/>
- 	</link>
- 	<link name="wheel_right">
-   		<visual>
-     			<geometry>
-       				<cylinder length="${length_wheel}" radius="${radius_wheel}"/>
-     			</geometry>
-			<!-- <origin rpy="0 1.5 0" xyz="-0.1 0.1 0"/> -->
-			<origin rpy="0 0 0" xyz="0 0 0"/>
-   			<material name="black"/>
-   		</visual>
-		<collision>
-			<geometry>
-       				<cylinder length="${length_wheel}" radius="${radius_wheel}"/>
-			</geometry>
-		</collision>
-		<xacro:default_inertial mass="1"/>
- 	</link>
- 	<link name="caster_wheel">
-   		<visual>
-     			<geometry>
-       				<sphere radius="${radius_wheel}"/>
-     			</geometry>
-			<!-- <origin rpy="0 1.5 0" xyz="0.1 -0.1 0"/> -->
-			<origin rpy="0 0 0" xyz="0 0 0"/>
-   			<material name="black"/>
-   		</visual>
-		<collision>
-			<geometry>
-       				<sphere radius="${radius_wheel}"/>
-			</geometry>
-		</collision>
-		<xacro:default_inertial mass="1"/>
- 	</link>
- <joint name="base_to_wheel_left" type="continuous">
-   <parent link="base_link"/>
-   <child link="wheel_left"/>
-   <origin rpy="-1.5707 0 0" xyz="-0.1 0.15 0"/>
-   <axis xyz="0 0 1" />
- </joint>
- <joint name="base_to_wheel_right" type="continuous">
-   <axis xyz="0 0 1" />
-   <anchor xyz="0 0 0" />
-   <limit effort="100" velocity="100" />
-   <parent link="base_link"/>
-   <child link="wheel_right"/>
-   <origin rpy="-1.5707 0 0" xyz="-0.1 -0.15 0"/>
-</joint>
- <joint name="base_to_caster_wheel" type="continuous">
-   <parent link="base_link"/>
-   <axis xyz="0 0 1" />
-   <child link="caster_wheel"/>
-   <origin rpy="-1.5707 0 0" xyz="0.1 0 0"/>
- </joint>
+<robot name="saturnbot" xmlns:xacro="http://ros.org/wiki/xacro">
+ <!-- base_link -->
+ <xacro:include filename="$(find saturnbot_description)/urdf/base/saturnbot_base.urdf.xacro" />
  <!-- camera_link -->
  <xacro:include filename="$(find saturnbot_description)/urdf/sensors/astra.urdf.xacro" />

File: robot/saturnbot_kinect.urdf.xacro (robot description, xacro)
@@ -3,123 +3,7 @@
     - 3d Sensor : kinect
 -->
-<robot name="turtlebot" xmlns:xacro="http://ros.org/wiki/xacro">
-  <xacro:property name="length_wheel" value="0.05" />
-	<xacro:property name="radius_wheel" value="0.05" />
-	<xacro:property name="camera_link" value="0.05" />
-  <xacro:property name="M_PI" value="3.1415926535897931" />
-	<xacro:macro name="default_inertial" params="mass">
-               <inertial>
-                       <mass value="${mass}" />
-                       <inertia ixx="1.0" ixy="0.0" ixz="0.0"
-                                iyy="1.0" iyz="0.0"
-                                izz="1.0" />
-               </inertial>
-	</xacro:macro>
-  <xacro:include filename="$(find saturnbot_description)/urdf/saturnbot_properties.urdf.xacro" />
-	<link name="base_footprint">
-   		<visual>
-			<geometry>
-      				<box size="0.001 0.001 0.001"/>
-     			</geometry>
-			<origin rpy="0 0 0" xyz="0 0 0"/>
-   		</visual>
-		<!--<xacro:default_inertial mass="0.0001"/>-->
- 	</link>
-	<gazebo reference="base_footprint">
-		<material>Gazebo/Green</material>
-		<turnGravityOff>false</turnGravityOff>
-	</gazebo>
-	<joint name="base_footprint_joint" type="fixed">
-		<origin xyz="0 0 0" />
-		<parent link="base_footprint" />
-		<child link="base_link" />
-	</joint>
-	<link name="base_link">
-   		<visual>
-			<geometry>
-      				<box size="0.2 .3 .1"/>
-     			</geometry>
-			<origin rpy="0 0 1.54" xyz="0 0 0.05"/>
-			<material name="white">
-				<color rgba="1 1 1 1"/>
-			</material>
-   		</visual>
-		<collision>
-			<geometry>
-       				<box size="0.2 .3 0.1"/>
-			</geometry>
-		</collision>
-		<xacro:default_inertial mass="10"/>
- 	</link>
- 	<link name="wheel_left">
-   		<visual>
-     			<geometry>
-       				<cylinder length="${length_wheel}" radius="${radius_wheel}"/>
-     			</geometry>
-			<!-- <origin rpy="0 1.5 0" xyz="0.1 0.1 0"/> -->
-			<origin rpy="0 0 0" xyz="0 0 0"/>
-   			<material name="black">
-				<color rgba="0 0 0 1"/>
-			</material>
-		</visual>
-		<collision>
-			<geometry>
-       				<cylinder length="${length_wheel}" radius="${radius_wheel}"/>
-			</geometry>
-		</collision>
-		<xacro:default_inertial mass="1"/>
- 	</link>
- 	<link name="wheel_right">
-   		<visual>
-     			<geometry>
-       				<cylinder length="${length_wheel}" radius="${radius_wheel}"/>
-     			</geometry>
-			<!-- <origin rpy="0 1.5 0" xyz="-0.1 0.1 0"/> -->
-			<origin rpy="0 0 0" xyz="0 0 0"/>
-   			<material name="black"/>
-   		</visual>
-		<collision>
-			<geometry>
-       				<cylinder length="${length_wheel}" radius="${radius_wheel}"/>
-			</geometry>
-		</collision>
-		<xacro:default_inertial mass="1"/>
- 	</link>
- 	<link name="caster_wheel">
-   		<visual>
-     			<geometry>
-       				<sphere radius="${radius_wheel}"/>
-     			</geometry>
-			<!-- <origin rpy="0 1.5 0" xyz="0.1 -0.1 0"/> -->
-			<origin rpy="0 0 0" xyz="0 0 0"/>
-   			<material name="black"/>
-   		</visual>
-		<collision>
-			<geometry>
-       				<sphere radius="${radius_wheel}"/>
-			</geometry>
-		</collision>
-		<xacro:default_inertial mass="1"/>
- 	</link>
- <joint name="base_to_wheel_left" type="continuous">
-   <parent link="base_link"/>
-   <child link="wheel_left"/>
-   <origin rpy="-1.5707 0 0" xyz="-0.1 0.15 0"/>
-   <axis xyz="0 0 1" />
- </joint>
- <joint name="base_to_wheel_right" type="continuous">
-   <axis xyz="0 0 1" />
-   <anchor xyz="0 0 0" />
-   <limit effort="100" velocity="100" />
-   <parent link="base_link"/>
-   <child link="wheel_right"/>
-   <origin rpy="-1.5707 0 0" xyz="-0.1 -0.15 0"/>
-</joint>
- <joint name="base_to_caster_wheel" type="continuous">
-   <parent link="base_link"/>
-   <axis xyz="0 0 1" />
-   <child link="caster_wheel"/>
-   <origin rpy="-1.5707 0 0" xyz="0.1 0 0"/>
- </joint>
+<robot name="saturnbot" xmlns:xacro="http://ros.org/wiki/xacro">
+ <!-- base_link -->
+ <xacro:include filename="$(find saturnbot_description)/urdf/base/saturnbot_base.urdf.xacro" />
  <!-- camera_link -->
  <xacro:include filename="$(find saturnbot_description)/urdf/sensors/kinect.urdf.xacro" />

File: urdf/saturnbot_gazebo.urdf.xacro (robot description, xacro)
@@ -1,4 +1,5 @@
 <?xml version="1.0"?>
 <robot name="saturnbot_gazebo" xmlns:xacro="http://ros.org/wiki/xacro">
+<xacro:property name="M_PI" value="3.1415926535897931" />
 <!-- materials -->
 <gazebo reference="base_link">
@@ -21,8 +22,8 @@
   <leftJoint>base_to_wheel_left</leftJoint>
   <rightJoint>base_to_wheel_right</rightJoint>
-  <wheelSeparation>4</wheelSeparation>
-  <wheelDiameter>0.1</wheelDiameter>
+  <wheelSeparation>0.166</wheelSeparation>
+  <wheelDiameter>0.065</wheelDiameter>
   <robotBaseFrame>base_footprint</robotBaseFrame>
-  <wheelTorque>5</wheelTorque>
+  <wheelTorque>0.35</wheelTorque>
   <topicName>cmd_vel</topicName>
   <commandTopic>cmd_vel</commandTopic>

File: urdf/saturnbot_properties.urdf.xacro (robot description, xacro)
@@ -19,7 +19,7 @@
      (currently in development and awaiting feedback)
    -->
-	<property name="cam_px" value="-0.1" />
+	<property name="cam_px" value="-0.04" />
 <!--	<property name="cam_py" value="-0.0125" /> Y varies for different configurations. get sets in sensors_urdf -->
-	<property name="cam_pz" value="0.25" />
+	<property name="cam_pz" value="0.12" />
 	<property name="cam_or" value="0" />
 	<property name="cam_op" value="0" />

File: urdf/sensors/astra.urdf.xacro (robot description, xacro)
@@ -6,5 +6,5 @@
   <xacro:property name="astra_depth_rel_rgb_py" value="0.0250" />
   <xacro:property name="astra_cam_rel_rgb_py"   value="-0.0125" />
-  <xacro:property name="astra_dae_display_scale"   value="1" />
+  <xacro:property name="astra_dae_display_scale"   value="0.5" />
   <!-- Parameterised in part by the values in saturnbot_properties.urdf.xacro -->
   <xacro:macro name="sensor_astra" params="parent">
