Commit message: update robot model and add launch file to view model

File: urdf/base/saturnbot_base.urdf.xacro (robot description, xacro)
@@ -36,5 +36,5 @@
       				<box size="0.119 0.185 0.05"/>
      			</geometry>
-			<origin rpy="0 0 1.54" xyz="0 0 0.021"/>
+			<origin rpy="0 0 1.54" xyz="0 0 0.046"/>
 			<material name="white">
 				<color rgba="1 1 1 1"/>
@@ -101,5 +101,5 @@
    <parent link="base_link"/>
    <child link="wheel_left"/>
-   <origin rpy="-1.5707 0 0" xyz="-0.071 0.083 0"/>
+   <origin rpy="-1.5707 0 0" xyz="-0.071 0.083 0.0325"/>
    <axis xyz="0 0 1" />
  </joint>
@@ -110,5 +110,5 @@
    <parent link="base_link"/>
    <child link="wheel_right"/>
-   <origin rpy="-1.5707 0 0" xyz="-0.071 -0.083 0"/>
+   <origin rpy="-1.5707 0 0" xyz="-0.071 -0.083 0.0325"/>
 </joint>
  <joint name="base_to_caster_wheel" type="continuous">
@@ -116,5 +116,5 @@
    <axis xyz="0 0 1" />
    <child link="caster_wheel"/>
-   <origin rpy="-1.5707 0 0" xyz="0.071 0 0"/>
+   <origin rpy="-1.5707 0 0" xyz="0.071 0 0.021"/>
  </joint>
 </robot>

File: urdf/saturnbot_properties.urdf.xacro (robot description, xacro)
@@ -21,5 +21,5 @@
 	<property name="cam_px" value="-0.04" />
 <!--	<property name="cam_py" value="-0.0125" /> Y varies for different configurations. get sets in sensors_urdf -->
-	<property name="cam_pz" value="0.12" />
+	<property name="cam_pz" value="0.20" />
 	<property name="cam_or" value="0" />
 	<property name="cam_op" value="0" />

File: urdf/sensors/astra.urdf.xacro (robot description, xacro)
@@ -9,9 +9,22 @@
   <!-- Parameterised in part by the values in saturnbot_properties.urdf.xacro -->
   <xacro:macro name="sensor_astra" params="parent">
-    <joint name="camera_joint" type="fixed">
+    <joint name="camera_rgb_joint" type="fixed">
       <origin xyz="${cam_px} ${astra_cam_py} ${cam_pz}"
               rpy="0 0 0"/>
       <parent link="${parent}"/>
-      <child link="camera_link" />
+      <child link="camera_rgb_frame" />
+    </joint>
+    <link name="camera_rgb_frame"/>
+    <joint name="camera_rgb_optical_joint" type="fixed">
+      <origin xyz="0 0 0" rpy="${-M_PI/2} 0 ${-M_PI/2}" />
+      <parent link="camera_rgb_frame" />
+      <child link="camera_rgb_optical_frame" />
+    </joint>
+    <link name="camera_rgb_optical_frame"/>
+    <joint name="camera_joint" type="fixed">
+      <origin xyz="0 ${astra_cam_rel_rgb_py} 0"
+              rpy="0 0 0"/>
+      <parent link="camera_rgb_frame"/>
+      <child link="camera_link"/>
     </joint>
     <link name="camera_link">
@@ -36,20 +49,7 @@
       </inertial>
     </link>
-    <joint name="camera_rgb_joint" type="fixed">
-      <origin xyz="0 ${astra_cam_rel_rgb_py} 0"
-              rpy="0 0 0"/>
-      <parent link="camera_link"/>
-      <child link="camera_rgb_frame"/>
-    </joint>
-    <link name="camera_rgb_frame"/>
-    <joint name="camera_rgb_optical_joint" type="fixed">
-      <origin xyz="0 0 0" rpy="${-M_PI/2} 0 ${-M_PI/2}" />
-      <parent link="camera_rgb_frame" />
-      <child link="camera_rgb_optical_frame" />
-    </joint>
-    <link name="camera_rgb_optical_frame"/>
     <joint name="camera_depth_joint" type="fixed">
       <origin xyz="0 ${astra_depth_rel_rgb_py} 0" rpy="0 0 0" />
-      <parent link="camera_link" />
+      <parent link="camera_rgb_frame" />
       <child link="camera_depth_frame" />
     </joint>
@@ -62,5 +62,5 @@
     <link name="camera_depth_optical_frame"/>
     <!-- RGBD sensor for simulation, same as Kinect -->
-    <saturnbot_sim_3dsensor/>
+    <turtlebot_sim_3dsensor/>
   </xacro:macro>
 </robot>

File: urdf/sensors/kinect.urdf.xacro (robot description, xacro)
@@ -5,34 +5,8 @@
   <!-- Parameterised in part by the values in saturnbot_properties.urdf.xacro -->
   <xacro:macro name="sensor_kinect" params="parent">
-    <joint name="camera_joint" type="fixed">
+    <joint name="camera_rgb_joint" type="fixed">
       <origin xyz="${cam_px} ${kinect_cam_py} ${cam_pz}" rpy="${cam_or} ${cam_op} ${cam_oy}"/>
       <parent link="${parent}"/>
-      <child link="camera_link" />
-    </joint>
-    <link name="camera_link">
-    <visual>
-     <origin xyz="0 0 0" rpy="0 0 ${M_PI/2}"/>
-      <geometry>
-       <mesh filename="package://saturnbot_description/meshes/sensors/kinect.dae"/>
-      </geometry>
-    </visual>
-    <collision>
-      <origin xyz="0.0 0.0 0.0" rpy="0 0 0"/>
-      <geometry>
-        <box size="0.07271 0.27794 0.073"/>
-      </geometry>
-    </collision>
-    <inertial>
-      <mass value="0.564" />
-      <origin xyz="0 0 0" />
-      <inertia ixx="0.003881243" ixy="0.0" ixz="0.0"
-               iyy="0.000498940" iyz="0.0"
-               izz="0.003879257" />
-    </inertial>
-  </link>
-    <joint name="camera_rgb_joint" type="fixed">
-      <origin xyz="-0.031 ${-kinect_cam_py} -0.016" rpy="0 0 0"/>
-      <parent link="camera_link"/>
-      <child link="camera_rgb_frame"/>
+      <child link="camera_rgb_frame" />
     </joint>
     <link name="camera_rgb_frame"/>
@@ -43,4 +17,30 @@
     </joint>
     <link name="camera_rgb_optical_frame"/>
+    <joint name="camera_joint" type="fixed">
+      <origin xyz="-0.031 ${-kinect_cam_py} -0.016" rpy="0 0 0"/>
+      <parent link="camera_rgb_frame"/>
+      <child link="camera_link"/>
+    </joint>
+      <link name="camera_link">
+      <visual>
+       <origin xyz="0 0 0" rpy="0 0 ${M_PI/2}"/>
+        <geometry>
+         <mesh filename="package://saturnbot_description/meshes/sensors/kinect.dae"/>
+        </geometry>
+      </visual>
+  	  <collision>
+        <origin xyz="0.0 0.0 0.0" rpy="0 0 0"/>
+  	    <geometry>
+  	      <box size="0.07271 0.27794 0.073"/>
+  	    </geometry>
+  	  </collision>
+      <inertial>
+        <mass value="0.564" />
+        <origin xyz="0 0 0" />
+        <inertia ixx="0.003881243" ixy="0.0" ixz="0.0"
+                 iyy="0.000498940" iyz="0.0"
+                 izz="0.003879257" />
+      </inertial>
+    </link>
     <!-- The fixed joints & links below are usually published by static_transformers launched by the OpenNi launch
          files. However, for Gazebo simulation we need them, so we add them here.
@@ -48,5 +48,5 @@
 	<joint name="camera_depth_joint" type="fixed">
 	  <origin xyz="0 ${2 * -kinect_cam_py} 0" rpy="0 0 0" />
-	  <parent link="camera_link" />
+	  <parent link="camera_rgb_frame" />
 	  <child link="camera_depth_frame" />
 	</joint>
