Commit message: complete astra robot model

File: urdf/sensors/astra.urdf.xacro (robot description, xacro)
@@ -1,5 +1,4 @@
 <?xml version="1.0"?>
 <robot name="sensor_astra" xmlns:xacro="http://ros.org/wiki/xacro">
-  <xacro:include filename="$(find saturnbot_description)/urdf/saturnbot_gazebo.urdf.xacro"/>
   <xacro:include filename="$(find saturnbot_description)/urdf/saturnbot_properties.urdf.xacro"/>
   <!-- Xacro properties -->
@@ -8,5 +7,4 @@
   <xacro:property name="astra_cam_rel_rgb_py"   value="-0.0125" />
   <xacro:property name="astra_dae_display_scale"   value="1" />
-  <xacro:property name="parent" value="base_link" />
   <!-- Parameterised in part by the values in saturnbot_properties.urdf.xacro -->
   <xacro:macro name="sensor_astra" params="parent">

Commit message: recover depth camera model

File: urdf/sensors/astra.urdf.xacro (robot description, xacro)
@@ -9,22 +9,9 @@
   <!-- Parameterised in part by the values in saturnbot_properties.urdf.xacro -->
   <xacro:macro name="sensor_astra" params="parent">
-    <joint name="camera_rgb_joint" type="fixed">
+    <joint name="camera_joint" type="fixed">
       <origin xyz="${cam_px} ${astra_cam_py} ${cam_pz}"
               rpy="0 0 0"/>
       <parent link="${parent}"/>
-      <child link="camera_rgb_frame" />
-    </joint>
-    <link name="camera_rgb_frame"/>
-    <joint name="camera_rgb_optical_joint" type="fixed">
-      <origin xyz="0 0 0" rpy="${-M_PI/2} 0 ${-M_PI/2}" />
-      <parent link="camera_rgb_frame" />
-      <child link="camera_rgb_optical_frame" />
-    </joint>
-    <link name="camera_rgb_optical_frame"/>
-    <joint name="camera_joint" type="fixed">
-      <origin xyz="0 ${astra_cam_rel_rgb_py} 0"
-              rpy="0 0 0"/>
-      <parent link="camera_rgb_frame"/>
-      <child link="camera_link"/>
+      <child link="camera_link" />
     </joint>
     <link name="camera_link">
@@ -49,7 +36,20 @@
       </inertial>
     </link>
+    <joint name="camera_rgb_joint" type="fixed">
+      <origin xyz="0 ${astra_cam_rel_rgb_py} 0"
+              rpy="0 0 0"/>
+      <parent link="camera_link"/>
+      <child link="camera_rgb_frame"/>
+    </joint>
+    <link name="camera_rgb_frame"/>
+    <joint name="camera_rgb_optical_joint" type="fixed">
+      <origin xyz="0 0 0" rpy="${-M_PI/2} 0 ${-M_PI/2}" />
+      <parent link="camera_rgb_frame" />
+      <child link="camera_rgb_optical_frame" />
+    </joint>
+    <link name="camera_rgb_optical_frame"/>
     <joint name="camera_depth_joint" type="fixed">
       <origin xyz="0 ${astra_depth_rel_rgb_py} 0" rpy="0 0 0" />
-      <parent link="camera_rgb_frame" />
+      <parent link="camera_link" />
       <child link="camera_depth_frame" />
     </joint>
@@ -62,5 +62,5 @@
     <link name="camera_depth_optical_frame"/>
     <!-- RGBD sensor for simulation, same as Kinect -->
-    <turtlebot_sim_3dsensor/>
+    <saturnbot_sim_3dsensor/>
   </xacro:macro>
 </robot>

File: urdf/sensors/kinect.urdf.xacro (robot description, xacro)
@@ -5,8 +5,34 @@
   <!-- Parameterised in part by the values in saturnbot_properties.urdf.xacro -->
   <xacro:macro name="sensor_kinect" params="parent">
-    <joint name="camera_rgb_joint" type="fixed">
+    <joint name="camera_joint" type="fixed">
       <origin xyz="${cam_px} ${kinect_cam_py} ${cam_pz}" rpy="${cam_or} ${cam_op} ${cam_oy}"/>
       <parent link="${parent}"/>
-      <child link="camera_rgb_frame" />
+      <child link="camera_link" />
+    </joint>
+    <link name="camera_link">
+    <visual>
+     <origin xyz="0 0 0" rpy="0 0 ${M_PI/2}"/>
+      <geometry>
+       <mesh filename="package://saturnbot_description/meshes/sensors/kinect.dae"/>
+      </geometry>
+    </visual>
+    <collision>
+      <origin xyz="0.0 0.0 0.0" rpy="0 0 0"/>
+      <geometry>
+        <box size="0.07271 0.27794 0.073"/>
+      </geometry>
+    </collision>
+    <inertial>
+      <mass value="0.564" />
+      <origin xyz="0 0 0" />
+      <inertia ixx="0.003881243" ixy="0.0" ixz="0.0"
+               iyy="0.000498940" iyz="0.0"
+               izz="0.003879257" />
+    </inertial>
+  </link>
+    <joint name="camera_rgb_joint" type="fixed">
+      <origin xyz="-0.031 ${-kinect_cam_py} -0.016" rpy="0 0 0"/>
+      <parent link="camera_link"/>
+      <child link="camera_rgb_frame"/>
     </joint>
     <link name="camera_rgb_frame"/>
@@ -17,30 +43,4 @@
     </joint>
     <link name="camera_rgb_optical_frame"/>
-    <joint name="camera_joint" type="fixed">
-      <origin xyz="-0.031 ${-kinect_cam_py} -0.016" rpy="0 0 0"/>
-      <parent link="camera_rgb_frame"/>
-      <child link="camera_link"/>
-    </joint>
-      <link name="camera_link">
-      <visual>
-       <origin xyz="0 0 0" rpy="0 0 ${M_PI/2}"/>
-        <geometry>
-         <mesh filename="package://saturnbot_description/meshes/sensors/kinect.dae"/>
-        </geometry>
-      </visual>
-  	  <collision>
-        <origin xyz="0.0 0.0 0.0" rpy="0 0 0"/>
-  	    <geometry>
-  	      <box size="0.07271 0.27794 0.073"/>
-  	    </geometry>
-  	  </collision>
-      <inertial>
-        <mass value="0.564" />
-        <origin xyz="0 0 0" />
-        <inertia ixx="0.003881243" ixy="0.0" ixz="0.0"
-                 iyy="0.000498940" iyz="0.0"
-                 izz="0.003879257" />
-      </inertial>
-    </link>
     <!-- The fixed joints & links below are usually published by static_transformers launched by the OpenNi launch
          files. However, for Gazebo simulation we need them, so we add them here.
@@ -48,5 +48,5 @@
 	<joint name="camera_depth_joint" type="fixed">
 	  <origin xyz="0 ${2 * -kinect_cam_py} 0" rpy="0 0 0" />
-	  <parent link="camera_rgb_frame" />
+	  <parent link="camera_link" />
 	  <child link="camera_depth_frame" />
 	</joint>
